Commit message: added kinect camera and rviz config

File: robots/jackal/jackal_description/urdf/jackal.urdf.xacro (robot description, xacro)
@@ -232,11 +232,11 @@
     <origin xyz="0 0 0.18" rpy="0 0 0" />
   </VLP-16>
-  <!-- Bring in simulation data for Gazebo.
-  <xacro:include filename="$(find jackal_description)/urdf/jackal.gazebo" />  -->
-  <!-- Optional standard accessories, including their simulation data. The rendering
-       of these into the final description is controlled by optenv variables, which
-       default each one to off.
-  <xacro:include filename="$(find jackal_description)/urdf/accessories.urdf.xacro" /> -->
-  <!-- Optional custom includes.
-  <xacro:include filename="$(optenv JACKAL_URDF_EXTRAS empty.urdf)" />  -->
+  <!-- add kinect camera -->
+  <xacro:include filename="$(find jackal_description)/urdf/sensors/kinect.urdf.xacro" />
+    <jackal_kinect/>
+    <joint name="kinect_mount_joint" type="fixed">
+      <origin xyz="0.1 0 0.05" rpy="0 0 0" />
+      <parent link="front_mount" />
+      <child link="kinect_mount" />
+    </joint>
 </robot>

File: robots/jackal/jackal_description/urdf/sensors.xacro (robot description, xacro)
@@ -24,19 +24,3 @@
     </sensor>
   </gazebo>
- <!--
-  <gazebo>
-    <plugin name="gps_controller" filename="libhector_gazebo_ros_gps.so">
-      <updateRate>40</updateRate>
-      <robotNamespace>/</robotNamespace>
-      <bodyName>navsat_link</bodyName>
-      <frameId>base_link</frameId>
-      <topicName>/navsat/fix</topicName>
-      <velocityTopicName>/navsat/vel</velocityTopicName>
-      <referenceLatitude>49.9</referenceLatitude>
-      <referenceLongitude>8.9</referenceLongitude>
-      <referenceHeading>0</referenceHeading>
-      <referenceAltitude>0</referenceAltitude>
-      <drift>0.0001 0.0001 0.0001</drift>
-    </plugin>
-  </gazebo> -->
 </robot>
